Commit message: update

File: urdf/hebi.urdf (robot description, URDF)
Before this commit: robot m6, 31 links, 30 joints
Links:
- link leg1__LAST_LINK: geometry collision box size=0.045000 0.047030 0.047030; collision box size=0.05850 0.04800 0.03650
- link leg2__LAST_LINK: geometry collision box size=0.045000 0.047030 0.047030; collision box size=0.05850 0.04800 0.03650
