Commit message: update

File: urdf/box.urdf (robot description, URDF)
Before this commit: robot box, 1 links, 0 joints
Links:
- link base_link: mass None -> 0.2

File: urdf/foundation.urdf (robot description, URDF)
Before this commit: robot foundation, 1 links, 0 joints
Links:
- removed link base_link
- added link link1, mass 1.8476; collision mesh filename=yuna_stl/object.STL; visual mesh filename=yuna_stl/object.STL

File: urdf/hebi-1.urdf (robot description, URDF)
Before this commit: robot m6, 31 links, 30 joints
Links:
- link leg1__LAST_LINK: geometry collision box size=0.045000 0.047030 0.047030; collision box size=0.05850 0.04800 0.03650
- link leg2__LAST_LINK: geometry collision box size=0.045000 0.047030 0.047030; collision box size=0.05850 0.04800 0.03650

File: urdf/hebi-2.urdf (robot description, URDF)
Before this commit: robot m6, 31 links, 30 joints
Links:
- link leg1__LAST_LINK: mass 0.229433 -> 0.3; geometry collision box size=0.045000 0.047030 0.047030; collision box size=0.05850 0.04800 0.03650
- link leg2__LAST_LINK: mass 0.229433 -> 0.3; geometry collision box size=0.045000 0.047030 0.047030; collision box size=0.05850 0.04800 0.03650
