Commit message: update

File: urdf/hebi-1.urdf (robot description, URDF)
Before this commit: robot m6, 31 links, 30 joints
Links:
- link leg1__LAST_LINK: mass 0.229433 -> 5
- link leg2__LAST_LINK: mass 0.229433 -> 5

File: urdf/hebi-2.urdf (robot description, URDF)
Before this commit: robot m6, 31 links, 30 joints
Links:
- link leg1__LAST_LINK: mass 0.3 -> 5
- link leg2__LAST_LINK: mass 0.3 -> 5

File: urdf/hebi.urdf (robot description, URDF)
Before this commit: robot m6, 31 links, 30 joints
Links:
- link leg1__LAST_LINK: mass 0.229433 -> 0.3
- link leg2__LAST_LINK: mass 0.229433 -> 0.3
